File: AlarmPCB/AlarmPCB.sch (KiCad schematic (older format))
At the start: 17 parts

Commit message: Updated Footprints
Parts:
- H1, H2, H3, H4: footprint MountingHole:MountingHole_3.2mm_M3 -> MountingHole:MountingHole_3.2mm_M3_DIN965_Pad
- RV1: footprint Potentiometer_THT:Potentiometer_ACP_CA6-H2,5_Horizontal -> digikey-footprints:Potentiometer_P120PK-Y25BR10K
Changed lines of the file:
@@
 EESchema Schematic File Version 4
+LIBS:AlarmPCB-cache
 EELAYER 30 0
 EELAYER END
@@
 F 0 "RV1" V 9300 3450 50  0000 R CNN
 F 1 "Contrast" H 9350 3550 50  0000 R CNN
-F 2 "Potentiometer_THT:Potentiometer_ACP_CA6-H2,5_Horizontal" H 9400 3400 50  0001 C CNN
+F 2 "digikey-footprints:Potentiometer_P120PK-Y25BR10K" H 9400 3400 50  0001 C CNN
 F 3 "~" H 9400 3400 50  0001 C CNN
 	1    9400 3400
@@
 F 0 "H1" H 6500 5796 50  0000 L CNN
 F 1 "MountingHole" H 6500 5705 50  0000 L CNN
-F 2 "MountingHole:MountingHole_3.2mm_M3" H 6400 5750 50  0001 C CNN
+F 2 "MountingHole:MountingHole_3.2mm_M3_DIN965_Pad" H 6400 5750 50  0001 C CNN
 F 3 "~" H 6400 5750 50  0001 C CNN
 	1    6400 5750
@@
 F 0 "H2" H 7250 5796 50  0000 L CNN
 F 1 "MountingHole" H 7250 5705 50  0000 L CNN
-F 2 "MountingHole:MountingHole_3.2mm_M3" H 7150 5750 50  0001 C CNN
+F 2 "MountingHole:MountingHole_3.2mm_M3_DIN965_Pad" H 7150 5750 50  0001 C CNN
 F 3 "~" H 7150 5750 50  0001 C CNN
 	1    7150 5750
@@
 F 0 "H3" H 8000 5796 50  0000 L CNN
 F 1 "MountingHole" H 8000 5705 50  0000 L CNN
-F 2 "MountingHole:MountingHole_3.2mm_M3" H 7900 5750 50  0001 C CNN
+F 2 "MountingHole:MountingHole_3.2mm_M3_DIN965_Pad" H 7900 5750 50  0001 C CNN
 F 3 "~" H 7900 5750 50  0001 C CNN
 	1    7900 5750
@@
 F 0 "H4" H 8750 5796 50  0000 L CNN
 F 1 "MountingHole" H 8750 5705 50  0000 L CNN
-F 2 "MountingHole:MountingHole_3.2mm_M3" H 8650 5750 50  0001 C CNN
+F 2 "MountingHole:MountingHole_3.2mm_M3_DIN965_Pad" H 8650 5750 50  0001 C CNN
 F 3 "~" H 8650 5750 50  0001 C CNN
 	1    8650 5750

Commit message: Revert "Updated Footprints"
This reverts commit dd3b0c72e674ffb159cfd3c8d42ceca2805da80f.
Parts:
- H1, H2, H3, H4: footprint MountingHole:MountingHole_3.2mm_M3_DIN965_Pad -> MountingHole:MountingHole_3.2mm_M3
- RV1: footprint digikey-footprints:Potentiometer_P120PK-Y25BR10K -> Potentiometer_THT:Potentiometer_ACP_CA6-H2,5_Horizontal
Changed lines of the file:
@@
 EESchema Schematic File Version 4
-LIBS:AlarmPCB-cache
 EELAYER 30 0
 EELAYER END
@@
 F 0 "RV1" V 9300 3450 50  0000 R CNN
 F 1 "Contrast" H 9350 3550 50  0000 R CNN
-F 2 "digikey-footprints:Potentiometer_P120PK-Y25BR10K" H 9400 3400 50  0001 C CNN
+F 2 "Potentiometer_THT:Potentiometer_ACP_CA6-H2,5_Horizontal" H 9400 3400 50  0001 C CNN
 F 3 "~" H 9400 3400 50  0001 C CNN
 	1    9400 3400
@@
 F 0 "H1" H 6500 5796 50  0000 L CNN
 F 1 "MountingHole" H 6500 5705 50  0000 L CNN
-F 2 "MountingHole:MountingHole_3.2mm_M3_DIN965_Pad" H 6400 5750 50  0001 C CNN
+F 2 "MountingHole:MountingHole_3.2mm_M3" H 6400 5750 50  0001 C CNN
 F 3 "~" H 6400 5750 50  0001 C CNN
 	1    6400 5750
@@
 F 0 "H2" H 7250 5796 50  0000 L CNN
 F 1 "MountingHole" H 7250 5705 50  0000 L CNN
-F 2 "MountingHole:MountingHole_3.2mm_M3_DIN965_Pad" H 7150 5750 50  0001 C CNN
+F 2 "MountingHole:MountingHole_3.2mm_M3" H 7150 5750 50  0001 C CNN
 F 3 "~" H 7150 5750 50  0001 C CNN
 	1    7150 5750
@@
 F 0 "H3" H 8000 5796 50  0000 L CNN
 F 1 "MountingHole" H 8000 5705 50  0000 L CNN
-F 2 "MountingHole:MountingHole_3.2mm_M3_DIN965_Pad" H 7900 5750 50  0001 C CNN
+F 2 "MountingHole:MountingHole_3.2mm_M3" H 7900 5750 50  0001 C CNN
 F 3 "~" H 7900 5750 50  0001 C CNN
 	1    7900 5750
@@
 F 0 "H4" H 8750 5796 50  0000 L CNN
 F 1 "MountingHole" H 8750 5705 50  0000 L CNN
-F 2 "MountingHole:MountingHole_3.2mm_M3_DIN965_Pad" H 8650 5750 50  0001 C CNN
+F 2 "MountingHole:MountingHole_3.2mm_M3" H 8650 5750 50  0001 C CNN
 F 3 "~" H 8650 5750 50  0001 C CNN
 	1    8650 5750
